File: hardware/controller/Nixie-Clock-Controller.kicad_pcb (KiCad board)
At the start: 2 copper layers, 228.6 x 69.8 mm, 67 parts, among them IC1 ESP32-DEVKITC-V4, IC2 74141, J1 9/12-35V DC in, J2 Nixies-Connector, J3 Input, J4 Output, J5 LEDs, J6 power_out, Q1 MPSA92, Q10 MPSA42, Q11 MPSA42, Q12 MPSA42, Q13 MPSA42, Q14 MPSA42, Q2 MPSA92, Q3 MPSA92, Q4 MPSA92, Q5 MPSA92, Q6 MPSA92, Q7 MPSA92, Q8 MPSA42, Q9 MPSA42, SW1 on/off, SW2 in voltage select, U1 L7805, U2 L7809, U3 NCH6300HV

Commit message: Improve labels
Parts:
- J1 - Vin: renamed from J1
- J2 - Nixies: renamed from J2; footprint nixie-clock:PinHeader_2x10_P2.54mm_Horizontal_with_Interlock -> Connector_PinHeader_2.54mm:PinHeader_2x10_P2.54mm_Vertical
- J3 - in: renamed from J3
- J4 - out: renamed from J4
- J5 - LED: renamed from J5
- J6 - Vout: renamed from J6
- SW1 - PWR: renamed from SW1
- SW2 - Vselect: renamed from SW2
- moved R2 5.08 mm to (76.2, 73.7)
- renumbered R4 to R10, R12 to R11, R13 to R12, R14 to R13, R15 to R14, R16 to R15, R17 to R16, R11 to R17, R19 to R18, R20 to R19, R21 to R20, R22 to R21, R23 to R22, R24 to R23, R18 to R24, R5 to R4, R6 to R5, R7 to R6, R8 to R7, R9 to R8, R10 to R9
