File: hardware/controller/Nixie-Clock-Controller.kicad_sch (KiCad schematic)
At the start: 67 parts, among them IC1 ESP32-DEVKITC-V4, IC2 74141, J1 9/12-35V DC in, J2 Nixies-Connector, J3 Input, J4 Output, J5 LEDs, J6 power_out, Q1 MPSA92, Q10 MPSA42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

Commit message: Improve labels
Parts:
- J2: footprint nixie-clock:PinHeader_2x10_P2.54mm_Horizontal_with_Interlock -> Connector_PinHeader_2.54mm:PinHeader_2x10_P2.54mm_Vertical
- renumbered R4 to R10, R12 to R11, R13 to R12, R14 to R13, R15 to R14, R16 to R15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
